File: KiCad/panama-keyboard.sch (KiCad schematic (older format))
At the start: 0 parts

Commit message: added switch matrix and mcu
Parts:
- added D? (x68): D_Small, symbol Device:D_Small
- added ESC1, ESC? (x18), Num1, Num? (x47): MX, symbol Keyboard:MX
- added SW?: Rotary_Encoder_Switch, symbol Device:Rotary_Encoder_Switch
- added SW? (x2): SW_Push, symbol Switch:SW_Push
- added U?: ATmega32A-PU, Package_DIP:DIP-40_W15.24mm, symbol MCU_Microchip_ATmega:ATmega32A-PU
Connections:
- new net: D?.2 (A), ESC1.2 (ROW)
- new net: D?.2 (A), Num1.2 (ROW)
- new net: D?.2 (A), Num?.2 (ROW) (x47)
- new net: D?.2 (A), ESC?.2 (ROW) (x18)
- new net: D?.1 (K), D?.1 (K), D?.1 (K), D?.1 (K), D?.1 (K), D?.1 (K), D?.1 (K), D?.1 (K), D?.1 (K), D?.1 (K), D?.1 (K)
- new net: U?.11 (GND), U?.31 (GND)
- new net col0: ESC1.1 (COL), ESC?.1 (COL), ESC?.1 (COL), ESC?.1 (COL), ESC?.1 (COL), ESC?.1 (COL), ESC?.1 (COL), ESC?.1 (COL), ESC?.1 (COL), ESC?.1 (COL), ESC?.1 (COL), ESC?.1 (COL), ESC?.1 (COL), ESC?.1 (COL), ESC?.1 (COL), ESC?.1 (COL), ESC?.1 (COL), ESC?.1 (COL), ESC?.1 (COL), Num1.1 (COL), Num?.1 (COL), Num?.1 (COL), Num?.1 (COL), Num?.1 (COL), Num?.1 (COL), Num?.1 (COL), Num?.1 (COL), Num?.1 (COL), Num?.1 (COL), Num?.1 (COL), Num?.1 (COL), Num?.1 (COL), Num?.1 (COL), Num?.1 (COL), Num?.1 (COL), Num?.1 (COL), Num?.1 (COL), Num?.1 (COL), Num?.1 (COL), Num?.1 (COL), Num?.1 (COL), Num?.1 (COL), Num?.1 (COL), Num?.1 (COL), Num?.1 (COL), Num?.1 (COL), Num?.1 (COL), Num?.1 (COL), Num?.1 (COL), Num?.1 (COL), Num?.1 (COL), Num?.1 (COL), Num?.1 (COL), Num?.1 (COL), Num?.1 (COL), Num?.1 (COL), Num?.1 (COL), Num?.1 (COL), Num?.1 (COL), Num?.1 (COL), Num?.1 (COL), Num?.1 (COL), Num?.1 (COL), Num?.1 (COL), Num?.1 (COL), Num?.1 (COL), Num?.1 (COL), SW?.S1
- new net enc-out: D?.2 (A), SW?.S2
- new net row0: D?.1 (K), D?.1 (K), D?.1 (K), D?.1 (K), D?.1 (K), D?.1 (K), D?.1 (K), D?.1 (K), D?.1 (K), D?.1 (K), D?.1 (K), D?.1 (K), D?.1 (K), D?.1 (K), D?.1 (K), D?.1 (K), D?.1 (K), D?.1 (K), D?.1 (K), D?.1 (K), D?.1 (K), D?.1 (K), D?.1 (K), D?.1 (K), D?.1 (K), D?.1 (K), D?.1 (K), D?.1 (K), D?.1 (K), D?.1 (K), D?.1 (K), D?.1 (K), D?.1 (K), D?.1 (K), D?.1 (K), D?.1 (K), D?.1 (K), D?.1 (K), D?.1 (K), D?.1 (K), D?.1 (K), D?.1 (K), D?.1 (K), D?.1 (K), D?.1 (K), D?.1 (K), D?.1 (K), D?.1 (K), D?.1 (K), D?.1 (K), D?.1 (K), D?.1 (K), D?.1 (K), D?.1 (K), D?.1 (K), D?.1 (K), D?.1 (K)
Other:
- note added: "BOOT"
- note added: "ENCODER"
- note added: "MCU"
- note added: "OLED"
- note added: "RESET"
- note added: "SWITCH MATRIX"
- note added: "UNDERGLOW"
- note added: "USB"

Commit message: schematic progress
Parts:
- added C1, C2: 22p, symbol Device:C_Small
- added C3, C4: 0.1u, symbol Device:C_Small
- added C5: 4.7u, symbol Device:CP_Small
- added D31, D32: 3.6V, symbol Device:D_Zener_Small
- added D?: WS2812B, LED_SMD:LED_WS2812B_PLCC4_5.0x5.0mm_P3.2mm, symbol LED:WS2812B
- added DS?: SSD1306-0.91-128x32, symbol Keyboard:SSD1306-0.91-128x32
- added F1: 500mA, symbol Device:Polyfuse_Small
- added J1: AVR-ISP-6, symbol Connector:AVR-ISP-6
- added J2: USB_C_Receptacle_USB2.0, symbol Connector:USB_C_Receptacle_USB2.0
- added R1, R2: 5.1k, symbol Device:R_Small
- added R3: 1.5k, symbol Device:R_Small
- added R4, R5: 68R, symbol Device:R_Small
- added R?: 10k, symbol Device:R_Small
- added Y1: Crystal, symbol Device:Crystal
- BOOT?: renamed from SW?; value SW_Push -> Boot
- ENC?: renamed from SW?; value Rotary_Encoder_Switch -> Encoder
- RESET?: renamed from SW?; value SW_Push -> Reset
- gave numbers to parts that had none: 134
Connections:
- net +5V: now reaches U1.10 (VCC)
- net +5V: now also U1.30 (AVCC), C3.1, C4.1, C5.1, DS?.2 (Vcc), F1.1, J1.2 (VCC), R3.1, R?.2
- net GND: now reaches U1.11 (GND), U1.31 (GND)
- net GND: now also BOOT?.2, ENC?.C, RESET?.2, C1.2, C2.2, C3.2, C4.2, C5.2, D31.2 (A), D32.2 (A), DS?.1 (GND), J1.6 (GND), J2.A1 (GND), J2.A12 (GND), J2.B1 (GND), J2.B12 (GND), J2.S1 (SHIELD), R1.1, R2.1
- net at U1.12 (XTAL2): now also C2.1, Y1.2
- net at U1.13 (XTAL1): now also C1.1, Y1.1
- net reset: now reaches U1.9 (~RESET)
- net reset: now also RESET?.1, J1.5 (~RST), R?.1
- net enc-A: now reaches ENC?.A
- net enc-B: now reaches ENC?.B
- net boot: now reaches BOOT?.1
- net enc-out renamed enc-sw-out
- new net: F1.2, J2.A4 (VBUS), J2.A9 (VBUS), J2.B4 (VBUS), J2.B9 (VBUS)
- new net: J2.A5 (CC1), R2.2
- new net: D31.1 (K), J2.A6 (D+), J2.B6 (D+), R5.2
- new net: D32.1 (K), J2.A7 (D-), J2.B7 (D-), R3.2, R4.2
- new net: J2.B5 (CC2), R1.2
- new net D+: R5.1
- new net D-: R4.1
- new net MISO: J1.1 (MISO)
- new net MOSI: J1.4 (MOSI)
- new net SCK: J1.3 (SCK)
- new net SCL: DS?.3 (SCL)
- new net SDA: DS?.4 (SDA)
- no-connect marks 0 -> 3
Other:
- note added: "ISP"
- moved on the sheet: BOOT?, ENC?, RESET?, U1

Commit message: schematic progress
Connections:
- net LED: now reaches D?.4 (DIN)
Changed lines of the file:
@@
 Text Notes 3700 3900 1    157  ~ 31
 SWITCH MATRIX
-Text Notes 2650 5550 0    157  ~ 31
-MCU
-Text Notes 5300 5600 0    157  ~ 31
-USB
 Text Notes 10200 5750 0    157  ~ 31
 UNDERGLOW
@@
 	1    0    0    -1
 $EndComp
-Text GLabel 12500 3000 3    50   Input ~ 10
+Text GLabel 12500 3000 3    50   Input ~ 0
 enc-sw-in
-Text GLabel 12300 3200 1    50   Input ~ 10
+Text GLabel 12300 3200 1    50   Input ~ 0
 enc-sw-out
-Text GLabel 8700 10200 2    50   Input ~ 10
+Text GLabel 8700 10200 2    50   Input ~ 0
 enc-sw-in
-Text GLabel 8700 10400 2    50   Input ~ 10
+Text GLabel 8700 10400 2    50   Input ~ 0
 enc-sw-out
 $Comp
@@
 	1    0    0    -1
 $EndComp
+Text Notes 5300 5600 0    157  ~ 31
+USB
+Text Notes 2650 5550 0    157  ~ 31
+MCU
+Text GLabel 10900 6400 0    50   Input ~ 0
+LED
+Text GLabel 3600 9400 2    50   Input ~ 0
+MISO
+Text GLabel 3600 9500 2    50   Input ~ 0
+MOSI
+Text GLabel 3600 9600 2    50   Input ~ 0
+SCK
+Text GLabel 3650 9150 2    50   Input ~ 0
+boot
+Text GLabel 3650 8900 2    50   Input ~ 0
+SCL
+Text GLabel 3650 8700 2    50   Input ~ 0
+SDA
+Text GLabel 3700 8500 2    50   Input ~ 0
+LED
+Text GLabel 3700 10050 2    50   Input ~ 0
+enc-A
+Text GLabel 3750 10250 2    50   Input ~ 0
+enc-B
+Text GLabel 3700 8250 2    50   Input ~ 0
+D-
+Text GLabel 3650 8050 2    50   Input ~ 0
+D+
 $EndSCHEMATC
