File: KiCad/panama-keyboard.kicad_pcb (KiCad board)
At the start: 2 copper layers, 170 parts, among them J1 MX, J2 USB_C_Receptacle_USB2.0, J3 AVR-ISP-6, K1 MX, M1 MX, P1 MX, Q1 MX, T1 MX, U1 MX, U2 ATmega32A-PU, X1 MX, Y1 MX, Y2 Crystal

Commit message: progree pcb
Parts:
- DS1: footprint OLED:PinHeader_1x04_P2.54mm_Vertical -> OLED:OLED_0.91in_128x32
- U2: footprint Package_DIP:DIP-40_W15.24mm -> Package_DIP:DIP-40_W15.24mm_Socket
- moved C2 307.3 mm to (481.0, 84.9)
- moved J2 307.3 mm to (495.7, 81.8)
- moved F2 266.3 mm to (515.9, 81.8)
- moved C6 218.6 mm to (161.1, 22.2)
- moved DS1 207.6 mm to (396.9, 139.7)
- moved D32 193.4 mm to (161.9, 138.1), turned to 270 degrees
- moved R6 191.8 mm to (495.3, 56.4)
- moved R4 188.1 mm to (496.6, 67.5)
- moved D61 187.0 mm to (168.3, 133.3), turned to 270 degrees
- moved D16 186.5 mm to (158.8, 140.5), turned to 270 degrees
- moved R2 181.6 mm to (508.8, 62.7)
- moved R5 176.2 mm to (510.4, 54.0)
- moved J3 174.3 mm to (464.3, 54.8)
- moved R7 168.1 mm to (481.8, 63.5)
- moved D48 165.3 mm to (190.5, 135.7), turned to 270 degrees
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
Commit message: pcb progress
Parts:
- moved D76 199.4 mm to (518.3, 71.4)
- moved R3 149.1 mm to (313.0, 64.5)
- moved U2 147.5 mm to (285.5, 119.5), turned to 90 degrees
- moved C6 140.7 mm to (293.2, 70.8)
- moved Y2 140.7 mm to (305.1, 77.2)
- moved C3 140.7 mm to (304.4, 90.8)
- moved C4 140.7 mm to (304.4, 94.8)
- moved C5 140.7 mm to (290.8, 78.0)
- moved J2 139.5 mm to (359.8, 113.2), turned to 180 degrees
- moved D75 118.0 mm to (525.5, 64.3)
- moved D30 98.4 mm to (358.8, 142.9), turned to 270 degrees
- moved D29 93.0 mm to (352.4, 138.1), turned to 270 degrees
- moved D70 84.5 mm to (368.3, 135.7), turned to 270 degrees
- moved D60 83.5 mm to (365.1, 138.1), turned to 270 degrees
- moved D45 80.3 mm to (361.9, 140.5), turned to 270 degrees
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Other:
- net class Default: trace_width 0.25 -> 0.254
- net class Power added: clearance 0.2, trace_width 0.381, via_dia 0.8, via_drill 0.4

Commit message: pcb progress
Parts:
- added REF**: MountingHole_3.2mm_M3, MountingHole:MountingHole_3.2mm_M3, F.Cu at (458.8, 256.4)
- added REF**: MountingHole_3.2mm_M3, MountingHole:MountingHole_3.2mm_M3, F.Cu at (149.2, 256.4)
- added REF**: MountingHole_3.2mm_M3, MountingHole:MountingHole_3.2mm_M3, F.Cu at (149.2, 124.6)
- added REF**: MountingHole_3.2mm_M3, MountingHole:MountingHole_3.2mm_M3, F.Cu at (458.8, 124.6)
- added REF**: MountingHole_3.2mm_M3, MountingHole:MountingHole_3.2mm_M3, F.Cu at (148.0, 196.8)
- moved D72 384.4 mm to (167.5, 328.6)
- moved D71 376.5 mm to (167.5, 308.0)
- moved D80 338.1 mm to (167.5, 291.3)
- moved D73 311.3 mm to (253.2, 328.6)
- moved D79 276.5 mm to (253.2, 291.3)
- moved D75 268.9 mm to (268.3, 142.9), turned to 270 degrees
- moved R5 261.6 mm to (263.2, 139.7)
- moved D76 257.0 mm to (271.5, 142.9), turned to 270 degrees
- moved R2 250.3 mm to (270.7, 139.7)
- moved F2 246.0 mm to (275.4, 133.3), turned to 180 degrees
- moved D82 238.8 mm to (354.8, 328.6)
- moved R6 231.1 mm to (281.0, 142.9), turned to 180 degrees
- moved C2 220.5 mm to (265.9, 133.3), turned to 180 degrees
- moved R4 220.2 mm to (285.8, 131.0), turned to 180 degrees
- moved R7 217.1 mm to (281.0, 146.1), turned to 180 degrees
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Other:
- board outline added: 319.1 x 167.5 mm

Commit message: pcb progress, back to 10 leds
Parts:
- removed REF** (x5): MountingHole_3.2mm_M3, MountingHole:MountingHole_3.2mm_M3
- D71, D72, D73, D74, D77, D78, D79, D80, D81, D82: moved to B.Cu
- moved D72 316.1 mm to (437.4, 164.0), turned to 90 degrees
- moved D81 276.7 mm to (168.8, 234.9)
- moved D71 247.0 mm to (358.0, 150.8), turned to 180 degrees
- moved D73 224.4 mm to (437.4, 200.4), turned to 90 degrees
- moved D77 172.9 mm to (254.0, 150.8), turned to 180 degrees
- moved D79 154.9 mm to (170.7, 160.2), turned to 270 degrees
- moved D29 147.4 mm to (400.8, 145.6)
- moved D30 147.4 mm to (404.0, 144.8)
- moved D69 147.4 mm to (397.7, 144.8)
- moved D60 147.3 mm to (407.2, 144.0)
- moved D44 147.3 mm to (394.5, 144.0)
- moved D13 147.2 mm to (391.3, 143.2)
- moved D46 146.8 mm to (410.4, 143.2)
- moved D82 134.9 mm to (257.7, 234.9)
- moved D15 127.8 mm to (381.8, 145.6)
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Other:
- board size 319.1 x 167.5 mm -> 319.1 x 141.3 mm

Commit message: pcb progress
Parts:
- moved D82 7.62 mm to (250.0, 234.9)
- moved D81 6.66 mm to (175.4, 234.9)
- moved D78 5.88 mm to (340.7, 234.9)
- moved D80 4.84 mm to (177.0, 194.9), turned to 270 degrees
- moved D72 3.66 mm to (437.4, 160.3)
- moved D79 3.66 mm to (170.7, 156.5)
- moved D73 1.83 mm to (437.4, 198.6)

Commit message: pcb progress
Parts:
- moved D2 20.8 mm to (171.4, 144.5)
- moved D61 18.8 mm to (155.6, 131.0)
- moved D3 17.8 mm to (177.8, 142.9)
- moved D63 17.4 mm to (165.1, 128.6)
- moved D5 17.1 mm to (193.7, 145.3)
- moved D33 17.1 mm to (168.3, 145.3)
- moved D37 17.1 mm to (190.5, 144.5)
- moved D48 17.1 mm to (165.1, 144.5)
- moved D20 16.7 mm to (193.7, 127.8)
- moved D21 16.7 mm to (200.0, 129.4)
- moved D52 16.7 mm to (190.5, 128.6)
- moved D38 15.6 mm to (196.8, 144.5)
- moved D62 15.4 mm to (161.9, 143.7)
- moved D51 15.2 mm to (184.2, 130.2)
- moved D53 15.2 mm to (196.8, 128.6)
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Routing:
- net col0: track 0.00 -> 250.5 mm, vias 0 -> 2
- net col1: track 0.00 -> 237.7 mm
- net col2: track 0.00 -> 222.5 mm
- net Net-(D53-Pad2): track 0.00 -> 150.0 mm
- net Net-(D64-Pad2): track 0.00 -> 140.4 mm
- net Net-(B1-Pad2): track 0.00 -> 137.4 mm
- net Net-(D63-Pad2): track 0.00 -> 127.4 mm
- net Net-(D51-Pad2): track 0.00 -> 122.8 mm
- net Net-(D38-Pad2): track 0.00 -> 115.8 mm
- net Net-(C1-Pad2): track 0.00 -> 112.4 mm
- net Net-(D61-Pad2): track 0.00 -> 108.3 mm
- net Net-(D49-Pad2): track 0.00 -> 106.5 mm
- net Net-(D36-Pad2): track 0.00 -> 104.4 mm
- net Net-(D37-Pad2): track 0.00 -> 103.6 mm
- net Net-(D62-Pad2): track 0.00 -> 99.6 mm
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
Commit message: pcb progress, moved switch matrix
Parts:
- D1, D10, D11, D12, D13, D14, D15, D16, D17, D18, D19, D2, D20, D21, D22, D23, D24, D25, D26, D27, D28, D29, D3, D30, D32, D33, D34, D35, D36, D37, D38, D39, D4, D40, D41, D42, D43, D44, D45, D46, D47, D48, D49, D5, D50, D51, D52, D53, D54, D55, D56, D57, D58, D59, D6, D60, D61, D62, D63, D64, D65, D66, D67, D68, D69, D7, D70, D8, D9: moved to B.Cu
- J3: footprint Connector_PinHeader_2.54mm:PinHeader_2x03_P2.54mm_Vertical -> Connector_PinHeader_2.54mm:PinHeader_1x06_P2.54mm_Horizontal
- moved D68 202.1 mm to (418.3, 242.1)
- moved D67 198.8 mm to (399.3, 242.1)
- moved D58 197.1 mm to (414.3, 223.0)
- moved D66 183.4 mm to (380.2, 242.1)
- moved D65 182.4 mm to (361.2, 242.1)
- moved D57 173.3 mm to (385.0, 223.0)
- moved D56 168.9 mm to (365.9, 223.0)
- moved D43 167.6 mm to (394.5, 204.0)
- moved D27 161.5 mm to (389.7, 184.9)
- moved D42 161.2 mm to (375.4, 204.0)
- moved D64 159.3 mm to (308.8, 242.1)
- moved D55 152.7 mm to (346.9, 223.0)
- moved D26 148.2 mm to (370.7, 184.9)
- moved D12 147.1 mm to (380.2, 165.9)
- moved D41 146.8 mm to (356.4, 204.0)
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Connections:
- ArrowDown1 pad 1: col8 -> col12
- ArrowLeft1 pad 1: col7 -> col11
- ArrowRight1 pad 1: col9 -> col13
- D10 pad 1: Net-(D10-Pad1) -> row0
- D11 pad 1: Net-(D10-Pad1) -> row0
- D12 pad 1: Net-(D10-Pad1) -> row0
- D13 pad 1: Net-(D10-Pad1) -> row0
- D14 pad 1: Net-(D10-Pad1) -> row0
- D15 pad 1: Net-(D10-Pad1) -> row0
- D5 pad 1: Net-(D10-Pad1) -> row0
- D6 pad 1: Net-(D10-Pad1) -> row0
- D7 pad 1: Net-(D10-Pad1) -> row0
- D77 pad 1: Net-(D77-Pad1) -> (no net)
- D8 pad 1: Net-(D10-Pad1) -> row0
- D9 pad 1: Net-(D10-Pad1) -> row0
- Func1 pad 1: col5 -> col9
- J2 pad A8: Net-(J2-PadA8) -> (no net)
- J2 pad B8: Net-(J2-PadB8) -> (no net)
- RAlt1 pad 1: col4 -> col8
- RCtrl1 pad 1: col6 -> col10
- U2 pad 19: Net-(U2-Pad19) -> (no net)
- U2 pad 32: Net-(U2-Pad32) -> (no net)
Routing:
- net row2: track 0.00 -> 350.4 mm
- net row0: track 0.00 -> 298.3 mm
- net row4: track 0.00 -> 285.0 mm
- net row1: track 0.00 -> 274.3 mm
- net row3: track 0.00 -> 261.4 mm
- net col0: track 250.5 -> 85.8 mm, vias 2 -> 0
- net col1: track 237.7 -> 94.1 mm
- net Net-(D53-Pad2): track 150.0 -> 17.8 mm
- net col2: track 222.5 -> 91.0 mm
- net Net-(D74-Pad1): track 0.00 -> 120.2 mm
- net Net-(B1-Pad2): track 137.4 -> 17.8 mm
- net col3: track 0.00 -> 115.6 mm
- net Net-(D63-Pad2): track 127.4 -> 20.2 mm
- net Net-(D64-Pad2): track 140.4 -> 34.5 mm
- net Net-(D51-Pad2): track 122.8 -> 17.8 mm
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Other:
- board size 319.1 x 141.3 mm -> 304.8 x 124.6 mm
- board text added: "+5V"
- board text added: "GND"
- board text added: "IN"
- board text added: "MISO"
- board text added: "MOSI"
- board text added: "RST"
- board text added: "SCK"

Commit message: logo added, PCB done
Parts:
- added G***: LOGO, LOGO:merciertech600, B.Cu at (255.4, 245.0)
- added G***: LOGO, LOGO:merciertech600, F.Cu at (254.0, 245.0)
- moved U2 51.1 mm to (323.9, 138.4), turned to 270 degrees
- moved R6 5.08 mm to (232.9, 152.4), turned to 180 degrees
- moved R7 5.08 mm to (232.9, 149.2), turned to 180 degrees
- moved D50 0.79 mm to (251.6, 222.2)
- moved D29 0.42 mm to (433.5, 184.5)
- moved D30 0.41 mm to (437.4, 184.5)
- moved BOOT1 0.32 mm to (198.8, 135.7)
- moved C5 0.25 mm to (326.8, 153.7)
- moved C3 0.22 mm to (296.2, 156.8)
- moved J3 0.18 mm to (178.1, 144.0)
- moved Y2 0.13 mm to (328.5, 143.6)
Routing:
- net col14: track 38.8 -> 205.9 mm, vias 0 -> 1
- net col0: track 85.8 -> 249.2 mm, vias 0 -> 2
- net col13: track 93.8 -> 243.2 mm, vias 0 -> 2
- net enc-A: track 0.00 -> 143.9 mm, vias 0 -> 3
- net enc-B: track 0.00 -> 142.1 mm, vias 0 -> 1
- net reset: track 0.00 -> 138.2 mm, vias 0 -> 3
- net MOSI: track 0.00 -> 134.3 mm, vias 0 -> 3
- net SCK: track 0.00 -> 134.3 mm, vias 0 -> 2
- net col1: track 94.1 -> 227.3 mm, vias 0 -> 2
- net col3: track 115.6 -> 229.9 mm
- net SCL: track 0.00 -> 112.3 mm, vias 0 -> 5
- net col2: track 91.0 -> 202.1 mm, vias 0 -> 1
- net SDA: track 0.00 -> 107.2 mm, vias 0 -> 3
- net row4: track 285.0 -> 387.3 mm, vias 0 -> 2
- net col12: track 92.0 -> 192.3 mm
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- added copper zone on F.Cu, net +5V
- added copper zone on B.Cu, net GND
Other:
- board text added: "<-LED START"
- board text added: "LED END"
- board text added: "PANAMA KEYBOARD v1.0 MERCIER TECHNOLOGIES"
